File: kicad_advance/pico_tracker.kicad_sch (KiCad schematic)
At the start: 42 parts, among them J1 MIDI_OUT, J10 DclassAMP, J11 CODEC_DIG, J12 CODEC_ANA, J13 LINE_IN, J14 PHONES, J15 MIC_MODULE, J16 FUEL_GAUGE, J2 MIDI_IN, J3 MIDI_IN_A_B_VCC, J4 MIDI_IN_A_B_DATA, J5 MIDI_OUT_A_B_VCC, J6 MIDI_OUT_A_B_DATA, J7 DISPLAY, J8 SDCARD, J9 KILL_SWITCH, SW1 LEFT, SW2 DOWN, SW3 RIGHT, SW4 UP, SW5 RT, SW6 B, SW7 A, SW8 LT, SW9 PLAY, U1 Pico, U2 6N138

Commit message: Advance-lite: widen codec header J12 to 1x9, reposition for ES8388 module mate
- J12 CODEC_ANA 6->9 pins (schematic); pins 7-9 carry the module line-out
  (LINEOUT_L/R/GND), unconnected on the mainboard.
- Move J12 on the PCB to (84.24, 91.84) so J11/J12 are 20.56mm apart, matching
  the ES8388 breakout module's two 1x9 edge headers (Digital-right/Analog-left).
- Add ES8388 module plan + schematic walkthrough docs.

Note: run Update PCB from Schematic to finalize J12's 6->9 footprint swap.
Parts:
- J12: footprint Connector_PinHeader_2.54mm:PinHeader_1x06_P2.54mm_Vertical -> Connector_PinHeader_2.54mm:PinHeader_1x09_P2.54mm_Vertical; symbol Connector:Conn_01x06_Female -> Connector:Conn_01x09_Female
- U1: value Pico -> Pico 2
Other:
- note added: "Keyboard matrix"
- note added: "MIDI I/O"
- moved on the sheet: D1, D10, D2, D3, D4, D5, D6, D7, D8, D9, J1, J11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
